Commit message: added simplified setup

File: src/arion_simulation/urdf/turtlebot3_waffle_pi.urdf.xacro (robot description, xacro)
@@ -1,159 +1,203 @@
 <?xml version="1.0" ?>
-<robot name="turtlebot3_waffle_pi" xmlns:xacro="http://www.ros.org/wiki/xacro">
-  <xacro:arg name="model" default="waffle_pi"/>
-  <!-- Base footprint -->
+<robot name="turtlebot3_waffle_pi" xmlns:xacro="http://ros.org/wiki/xacro">
   <link name="base_footprint"/>
-  <joint name="base_footprint_joint" type="revolute">
-    <origin xyz="0 0 0" rpy="0 0 0"/>
+  <joint name="base_joint" type="fixed">
+    <parent link="base_footprint"/>
     <child link="base_link"/>
-    <parent link="base_footprint"/>
+    <origin xyz="0.0 0.0 0.010" rpy="0 0 0"/>
+  </joint>
+  <link name="base_link">
+    <visual>
+      <origin xyz="-0.064 0 0.0" rpy="0 0 0"/>
+      <geometry>
+        <box size="0.265 0.265 0.089"/>
+      </geometry>
+      <material name="dark_grey">
+          <color rgba="0.2 0.2 0.2 1.0"/>
+      </material>
+    </visual>
+    <collision>
+      <origin xyz="-0.064 0 0.047" rpy="0 0 0"/>
+      <geometry>
+        <box size="0.265 0.265 0.089"/>
+      </geometry>
+    </collision>
+    <inertial>
+      <origin xyz="0 0 0" rpy="0 0 0"/>
+      <mass value="1.3729096"/>
+      <inertia ixx="0.0087002718" ixy="-0.000047576583" ixz="0.00011160499"
+               iyy="0.0086195418" iyz="-0.0000035422299"
+               izz="0.014653337" />
+    </inertial>
+  </link>
+  <joint name="wheel_left_joint" type="continuous">
+    <parent link="base_link"/>
+    <child link="wheel_left_link"/>
+    <origin xyz="0.0 0.144 0.023" rpy="-1.57 0 0"/>
     <axis xyz="0 0 1"/>
-    <limit effort="150" velocity="3.0" lower="-1.57" upper="1.57"/>
-  </joint>
-  <!-- Base link -->
-  <link name="base_link">
-    <visual>
-      <origin xyz="0 0 0.032" rpy="0 0 0"/>
-      <geometry>
-        <box size="0.265 0.265 0.086"/>
-      </geometry>
-      <material name="darkgray">
-        <color rgba="0.2 0.2 0.2 1.0"/>
+  </joint>
+  <link name="wheel_left_link">
+    <visual>
+      <origin xyz="0 0 0" rpy="1.57 0 0"/>
+      <geometry>
+        <cylinder length="0.018" radius="0.033"/>
+      </geometry>
+      <material name="black">
+          <color rgba="0 0 0 1"/>
       </material>
     </visual>
     <collision>
-      <origin xyz="0 0 0.032" rpy="0 0 0"/>
-      <geometry>
-        <box size="0.265 0.265 0.086"/>
-      </geometry>
-    </collision>
-    <inertial>
-      <mass value="1.3"/>
-      <origin xyz="0 0 0.032" rpy="0 0 0"/>
-      <inertia ixx="0.001" iyy="0.001" izz="0.001" ixy="0" ixz="0" iyz="0"/>
-    </inertial>
-  </link>
-  <!-- Left wheel -->
-  <joint name="wheel_left_joint" type="continuous">
-    <parent link="base_link"/>
-    <child link="wheel_left_link"/>
-    <origin xyz="0 0.08 0" rpy="-1.57 0 0"/>
+      <origin xyz="0 0 0" rpy="0 0 0"/>
+      <geometry>
+        <cylinder length="0.018" radius="0.033"/>
+      </geometry>
+    </collision>
+    <inertial>
+      <origin xyz="0 0 0" />
+      <mass value="0.028498940" />
+      <inertia ixx="0.000011175580" ixy="-0.000000000042269582" ixz="-0.000000000028800741"
+               iyy="0.000011192413" iyz="-0.0000000000011556285"
+               izz="0.000020712558" />
+    </inertial>
+  </link>
+  <joint name="wheel_right_joint" type="continuous">
+    <parent link="base_link"/>
+    <child link="wheel_right_link"/>
+    <origin xyz="0.0 -0.144 0.023" rpy="-1.57 0 0"/>
     <axis xyz="0 0 1"/>
-    <limit effort="100" velocity="6.28"/>
-  </joint>
-  <link name="wheel_left_link">
+  </joint>
+  <link name="wheel_right_link">
     <visual>
       <origin xyz="0 0 0" rpy="1.57 0 0"/>
       <geometry>
-        <cylinder length="0.025" radius="0.033"/>
+        <cylinder length="0.018" radius="0.033"/>
       </geometry>
       <material name="black">
-        <color rgba="0 0 0 1.0"/>
+          <color rgba="0 0 0 1"/>
       </material>
     </visual>
     <collision>
-      <origin xyz="0 0 0" rpy="1.57 0 0"/>
-      <geometry>
-        <cylinder length="0.025" radius="0.033"/>
-      </geometry>
-    </collision>
-    <inertial>
-      <mass value="0.1"/>
-      <origin xyz="0 0 0" rpy="1.57 0 0"/>
-      <inertia ixx="0.00001" iyy="0.00001" izz="0.00001" ixy="0" ixz="0" iyz="0"/>
-    </inertial>
-  </link>
-  <!-- Right wheel -->
-  <joint name="wheel_right_joint" type="continuous">
-    <parent link="base_link"/>
-    <child link="wheel_right_link"/>
-    <origin xyz="0 -0.08 0" rpy="-1.57 0 0"/>
-    <axis xyz="0 0 1"/>
-    <limit effort="100" velocity="6.28"/>
-  </joint>
-  <link name="wheel_right_link">
-    <visual>
-      <origin xyz="0 0 0" rpy="1.57 0 0"/>
-      <geometry>
-        <cylinder length="0.025" radius="0.033"/>
-      </geometry>
-      <material name="black">
-        <color rgba="0 0 0 1.0"/>
-      </material>
-    </visual>
-    <collision>
-      <origin xyz="0 0 0" rpy="1.57 0 0"/>
-      <geometry>
-        <cylinder length="0.025" radius="0.033"/>
-      </geometry>
-    </collision>
-    <inertial>
-      <mass value="0.1"/>
-      <origin xyz="0 0 0" rpy="1.57 0 0"/>
-      <inertia ixx="0.00001" iyy="0.00001" izz="0.00001" ixy="0" ixz="0" iyz="0"/>
-    </inertial>
-  </link>
-  <!-- Caster wheel -->
-  <joint name="caster_joint" type="fixed">
-    <parent link="base_link"/>
-    <child link="caster_link"/>
-    <origin xyz="-0.069 0 -0.004" rpy="-1.57 0 0"/>
-  </joint>
-  <link name="caster_link">
-    <visual>
-      <origin xyz="0 0 0" rpy="1.57 0 0"/>
-      <geometry>
-        <sphere radius="0.016"/>
-      </geometry>
-      <material name="black">
-        <color rgba="0 0 0 1.0"/>
-      </material>
-    </visual>
-    <collision>
-      <origin xyz="0 0 0" rpy="1.57 0 0"/>
-      <geometry>
-        <sphere radius="0.016"/>
-      </geometry>
-    </collision>
-    <inertial>
-      <mass value="0.05"/>
-      <origin xyz="0 0 0" rpy="1.57 0 0"/>
-      <inertia ixx="0.000001" iyy="0.000001" izz="0.000001" ixy="0" ixz="0" iyz="0"/>
-    </inertial>
-  </link>
-  <!-- Lidar sensor mounting -->
-  <joint name="lidar_joint" type="fixed">
-    <parent link="base_link"/>
-    <child link="lidar_link"/>
-    <origin xyz="0 0 0.068" rpy="0 0 0"/>
-  </joint>
-  <link name="lidar_link">
-    <visual>
-      <origin xyz="0 0 0" rpy="0 0 0"/>
-      <geometry>
-        <cylinder length="0.04" radius="0.04"/>
-      </geometry>
-      <material name="red">
-        <color rgba="1.0 0 0 1.0"/>
-      </material>
-    </visual>
-    <collision>
-      <origin xyz="0 0 0" rpy="0 0 0"/>
-      <geometry>
-        <cylinder length="0.04" radius="0.04"/>
-      </geometry>
-    </collision>
-    <inertial>
-      <mass value="0.125"/>
-      <origin xyz="0 0 0" rpy="0 0 0"/>
-      <inertia ixx="0.000001" iyy="0.000001" izz="0.000001" ixy="0" ixz="0" iyz="0"/>
-    </inertial>
-  </link>
-  <!-- IMU link (simulated) -->
-  <joint name="imu_joint" type="fixed">
-    <parent link="base_link"/>
-    <child link="imu_link"/>
-    <origin xyz="0 0 0.032" rpy="0 0 0"/>
-  </joint>
-  <link name="imu_link"/>
+      <origin xyz="0 0 0" rpy="0 0 0"/>
+      <geometry>
+        <cylinder length="0.018" radius="0.033"/>
+      </geometry>
+    </collision>
+    <inertial>
+      <origin xyz="0 0 0" />
+      <mass value="0.028498940" />
+      <inertia ixx="0.000011175580" ixy="-0.000000000042269582" ixz="-0.000000000028800741"
+               iyy="0.000011192413" iyz="-0.0000000000011556285"
+               izz="0.000020712558" />
+    </inertial>
+  </link>
+  <joint name="caster_back_right_joint" type="fixed">
+    <parent link="base_link"/>
+    <child link="caster_back_right_link"/>
+    <origin xyz="-0.177 -0.064 -0.004" rpy="-1.57 0 0"/>
+  </joint>
+  <link name="caster_back_right_link">
+    <collision>
+      <origin xyz="0 0.001 0" rpy="0 0 0"/>
+      <geometry>
+        <box size="0.030 0.009 0.020"/>
+      </geometry>
+    </collision>
+    <inertial>
+      <origin xyz="0 0 0" />
+      <mass value="0.005" />
+      <inertia ixx="0.001" ixy="0.0" ixz="0.0"
+               iyy="0.001" iyz="0.0"
+               izz="0.001" />
+    </inertial>
+  </link>
+  <joint name="caster_back_left_joint" type="fixed">
+    <parent link="base_link"/>
+    <child link="caster_back_left_link"/>
+    <origin xyz="-0.177 0.064 -0.004" rpy="-1.57 0 0"/>
+  </joint>
+  <link name="caster_back_left_link">
+    <collision>
+      <origin xyz="0 0.001 0" rpy="0 0 0"/>
+      <geometry>
+        <box size="0.030 0.009 0.020"/>
+      </geometry>
+    </collision>
+    <inertial>
+      <origin xyz="0 0 0" />
+      <mass value="0.005" />
+      <inertia ixx="0.001" ixy="0.0" ixz="0.0"
+               iyy="0.001" iyz="0.0"
+               izz="0.001" />
+    </inertial>
+  </link>
+  <joint name="scan_joint" type="fixed">
+    <parent link="base_link"/>
+    <child link="base_scan"/>
+    <origin xyz="-0.064 0 0.122" rpy="0 0 0"/>
+  </joint>
+  <link name="base_scan">
+    <visual>
+      <origin xyz="0 0 0" rpy="0 0 0"/>
+      <geometry>
+        <cylinder length="0.0315" radius="0.055"/>
+      </geometry>
+      <material name="dark_grey"/>
+    </visual>
+    <collision>
+      <origin xyz="0 0 0" rpy="0 0 0"/>
+      <geometry>
+        <cylinder length="0.0315" radius="0.055"/>
+      </geometry>
+    </collision>
+    <inertial>
+      <mass value="0.114" />
+      <origin xyz="0 0 0" />
+      <inertia ixx="0.001" ixy="0.0" ixz="0.0"
+               iyy="0.001" iyz="0.0"
+               izz="0.001" />
+    </inertial>
+  </link>
+  <gazebo>
+    <plugin filename="ign_ros2_control-system" name="ign_ros2_control::IgnitionROS2ControlPlugin">
+      <parameters>$(find arion_simulation)/config/ros2_control.yaml</parameters>
+    </plugin>
+    <plugin filename="ignition-gazebo-diff-drive-system" name="ignition::gazebo::systems::DiffDrive">
+      <left_joint>wheel_left_joint</left_joint>
+      <right_joint>wheel_right_joint</right_joint>
+      <wheel_separation>0.287</wheel_separation>
+      <wheel_radius>0.033</wheel_radius>
+      <odom_publish_frequency>30</odom_publish_frequency>
+      <topic>cmd_vel</topic>
+      <odom_topic>odom</odom_topic>
+      <tf_topic>tf</tf_topic>
+      <frame_id>odom</frame_id>
+      <child_frame_id>base_footprint</child_frame_id>
+    </plugin>
+    <plugin filename="ignition-gazebo-joint-state-publisher-system" name="ignition::gazebo::systems::JointStatePublisher">
+      <topic>joint_states</topic>
+    </plugin>
+  </gazebo>
+  <gazebo reference="base_scan">
+    <sensor name="hls_lfcd_lds" type="gpu_lidar">
+      <topic>scan</topic>
+      <update_rate>5</update_rate>
+      <ray>
+        <scan>
+          <horizontal>
+            <samples>360</samples>
+            <resolution>1</resolution>
+            <min_angle>0.0</min_angle>
+            <max_angle>6.28319</max_angle>
+          </horizontal>
+        </scan>
+        <range>
+          <min>0.120</min>
+          <max>3.5</max>
+          <resolution>0.015</resolution>
+        </range>
+      </ray>
+      <always_on>1</always_on>
+      <visualize>true</visualize>
+    </sensor>
+  </gazebo>
 </robot>

Commit message: udpated simulator objects

File: src/arion_simulation/urdf/turtlebot3_waffle_pi.urdf.xacro (robot description, xacro)
@@ -13,6 +13,6 @@
         <box size="0.265 0.265 0.089"/>
       </geometry>
-      <material name="dark_grey">
-          <color rgba="0.2 0.2 0.2 1.0"/>
+      <material name="Orange">
+          <color rgba="1.0 0.5 0.0 1.0"/>
       </material>
     </visual>
